File: uC3Moy.sch (KiCad schematic (older format))
At the start: 17 parts

Commit message: Commit subiendo el diseño principal
Parts:
- removed C? (x2): C, symbol C
- removed C? (x2): CP1, symbol CP1
- removed P?: CONN_2, symbol CONN_2
- removed R? (x2): R, symbol R
- added C1, C2: CAPAPOL, ~, symbol CAPAPOL
- added C3, C4, C5: C, ~, symbol C
- added D1: LED, ~, symbol LED
- added D2: DIODE, ~, symbol DIODE
- added J1: JACK_INT, symbol JACK_INT
- added J2: JACK, symbol JACK
- added PWR-/+1: CONN_2, symbol CONN_2
- added R1, R8, R9: R, ~, symbol R
- added U2, U3: TLE2426, symbol TLE2426
- C6, C7: renamed from C?; value C -> 1 uF
- U1: renamed from U?; value TL072 -> OPA2132
- gave numbers to parts that had none: 6
Connections:
- net labels added: +6V, -6V
- net labels removed: +5V, -5V
- wire segments 62 -> 57
- no-connect marks 0 -> 2
Other:
- moved on the sheet: C6, R2, R4, R6, U1A
