File: KiCadFiles/uC3Moy.sch (KiCad schematic (older format))
At the start: 24 parts, among them J1 JACK_INT, J2 JACK, U1 OPA2132, U2 TLE2426, U3 TLE2426

Commit message: Savepoint
Parts:
- removed C1, C2: CAPAPOL, ~, symbol CAPAPOL
- removed C3: C, ~, symbol C
- removed D1: LED, ~, symbol LED
- removed D2: DIODE, ~, symbol DIODE
- removed R1: R, ~, symbol R
- removed U3: TLE2426, symbol TLE2426
- added C5, C6: CP, Capacitors_ThroughHole:C_Radial_D5_L6_P2.5, symbol CP
- added R7, R8: R, Discret:R1, symbol R
- C1: renamed from C6; footprint (none) -> Capacitors_ThroughHole:C_Rect_L7_W2.5_P5
- C2: renamed from C7; footprint (none) -> Capacitors_ThroughHole:C_Rect_L7_W2.5_P5
- C3: renamed from C4; footprint ~ -> Capacitors_ThroughHole:C_Rect_L4_W2.5_P2.5
- C4: renamed from C5; footprint ~ -> Capacitors_ThroughHole:C_Rect_L4_W2.5_P2.5
- J1: footprint (none) -> uC3Moy:jackint
- J2: footprint (none) -> uC3Moy:jack
- PWR-/+1: footprint (none) -> Pin_Headers:Pin_Header_Straight_1x02
- R1: renamed from R2; footprint (none) -> Discret:R1
- R10: renamed from R8; footprint ~ -> Discret:R1
- R2: renamed from R3; footprint (none) -> Discret:R1
- R3: renamed from R4; footprint (none) -> Discret:R1
- R4: renamed from R5; footprint (none) -> Discret:R1
- R5: renamed from R6; footprint (none) -> Discret:R1
- R6: renamed from R7; footprint (none) -> Discret:R1
- R9: footprint ~ -> Discret:R1
- U1: footprint (none) -> uC3Moy:DIP-8_W7.62mm_jorfru
- U2: footprint (none) -> Housings_TO-92:TO-92_Inline_Wide
Connections:
- net +6V: now also C5.1, R7.2
- net -6V: now also C6.2, R8.2
- net GND: now also C5.2, C6.1, R7.1, R8.1
Other:
- moved on the sheet: C3, C4, U2
